File: badge/badge.kicad_pcb (KiCad board)
At the start: 2 copper layers, 60 x 95.5 mm, 6 parts, among them U1 NT3H2111W0FHKH

Commit message: boop
Parts:
- moved G*** 84.4 mm to (164.2, 110.2)
- moved 2 54.5 mm to (164.9, 67.1)
- moved U1 47.3 mm to (138.4, 58.8), turned to 180 degrees
- moved LED1 47.2 mm to (142.2, 52.3)
- moved C1 47.1 mm to (138.4, 56.7)
- moved R1 46.9 mm to (138.5, 55.0)
Routing:
- net U1_8: track 0.00 -> 39.1 mm, vias 0 -> 2
- net U1_1: track 0.00 -> 28.5 mm, vias 0 -> 1
- net U1_2: track 0.00 -> 9.55 mm
- net U1_6: track 0.00 -> 4.83 mm
- net LED1_1: track 0.00 -> 3.48 mm
Other:
- outline, holes or cut-outs redrawn
